File: a-to-m/a-to-m.sch (KiCad schematic (older format))
At the start: 1 part, among them U1 ESP8285

Commit message: Use generic QFN32 package
Parts:
- U1: footprint Package_DFN_QFN:QFN-32-1EP_5x5mm_P0.5mm_EP3.45x3.45mm -> Package_DFN_QFN:QFN-32-1EP_5x5mm_P0.5mm_EP3.7x3.7mm
Changed lines of the file:
@@
 F 0 "U1" H 5600 2411 50  0000 C CNN
 F 1 "ESP8285" H 5600 2320 50  0000 C CNN
-F 2 "Package_DFN_QFN:QFN-32-1EP_5x5mm_P0.5mm_EP3.45x3.45mm" H 5600 2300 50  0001 C CNN
+F 2 "Package_DFN_QFN:QFN-32-1EP_5x5mm_P0.5mm_EP3.7x3.7mm" H 5600 2300 50  0001 C CNN
 F 3 "http://espressif.com/sites/default/files/documentation/0a-esp8266ex_datasheet_en.pdf" H 5700 2300 50  0001 C CNN
 	1    5600 3600
